File: hw/kicad/usb_pwrmon.sch (KiCad schematic (older format))
At the start: 0 parts

Commit message: - add pic & lcd panel components
Parts:
- added J?: LCD-S401M16KR, symbol LCD-S401M16KR
- added U?: PIC16LF1933-I/SS, symbol PIC16LF1933-I/SS
Connections:
- net labels added: COM0, COM1, COM2, COM3, SEG0, SEG1, SEG2, SEG3, SEG4, SEG5, SEG6, SEG7
- wire segments 0 -> 22
Changed lines of the file:
@@
-EESchema Schematic File Version 2  date 1/22/2013 8:34:43 PM
+EESchema Schematic File Version 2  date 1/22/2013 9:40:15 PM
 LIBS:power
 LIBS:device
@@
 LIBS:contrib
 LIBS:valves
-EELAYER 43  0
+LIBS:usb_pwrmon
+LIBS:usb_pwrmon-cache
+EELAYER 25  0
 EELAYER END
 $Descr A4 11700 8267
@@
 Comment4 ""
 $EndDescr
+Wire Wire Line
+	6700 3300 6550 3300
+Wire Wire Line
+	4550 4800 4400 4800
+Wire Wire Line
+	4550 4200 4400 4200
+Wire Wire Line
+	4550 3750 4400 3750
+Wire Wire Line
+	4550 3450 4400 3450
+Wire Wire Line
+	7700 4700 7550 4700
+Wire Wire Line
+	7700 4400 7550 4400
+Wire Wire Line
+	7700 4100 7550 4100
+Wire Wire Line
+	7700 3800 7550 3800
+Wire Wire Line
+	7700 3500 7550 3500
+Wire Wire Line
+	7700 3200 7550 3200
+Wire Wire Line
+	7550 3050 7700 3050
+Wire Wire Line
+	7550 3350 7700 3350
+Wire Wire Line
+	7550 3650 7700 3650
+Wire Wire Line
+	7550 3950 7700 3950
+Wire Wire Line
+	7550 4250 7700 4250
+Wire Wire Line
+	7550 4550 7700 4550
+Wire Wire Line
+	4400 3300 4550 3300
+Wire Wire Line
+	4400 3600 4550 3600
+Wire Wire Line
+	4400 3900 4550 3900
+Wire Wire Line
+	4400 4350 4550 4350
+Wire Wire Line
+	4400 4950 4550 4950
+Text GLabel 4400 3300 0    60   Input ~ 0
+SEG7
+Text GLabel 4400 4950 0    60   Input ~ 0
+SEG6
+Text GLabel 4400 3900 0    60   Input ~ 0
+SEG5
+Text GLabel 4400 3750 0    60   Input ~ 0
+SEG4
+Text GLabel 4400 4800 0    60   Input ~ 0
+SEG3
+Text GLabel 4400 4200 0    60   Input ~ 0
+SEG2
+Text GLabel 4400 4350 0    60   Input ~ 0
+SEG1
+Text GLabel 6700 4050 2    60   Input ~ 0
+SEG0
+Text GLabel 4400 3600 0    60   Input ~ 0
+COM3
+Text GLabel 4400 3450 0    60   Input ~ 0
+COM2
+Text GLabel 6700 3300 2    60   Input ~ 0
+COM1
+Text GLabel 6700 3450 2    60   Input ~ 0
+COM0
+Text GLabel 7550 4700 0    60   Input ~ 0
+SEG7
+Text GLabel 7550 4550 0    60   Input ~ 0
+SEG6
+Text GLabel 7550 4400 0    60   Input ~ 0
+SEG5
+Text GLabel 7550 4250 0    60   Input ~ 0
+SEG4
+Text GLabel 7550 4100 0    60   Input ~ 0
+SEG3
+Text GLabel 7550 3950 0    60   Input ~ 0
+SEG2
+Text GLabel 7550 3800 0    60   Input ~ 0
+SEG1
+Text GLabel 7550 3650 0    60   Input ~ 0
+SEG0
+Text GLabel 7550 3500 0    60   Input ~ 0
+COM3
+Text GLabel 7550 3350 0    60   Input ~ 0
+COM2
+Text GLabel 7550 3200 0    60   Input ~ 0
+COM1
+Text GLabel 7550 3050 0    60   Input ~ 0
+COM0
+$Comp
+L LCD-S401M16KR J?
+U 1 1 50FF4B2C
+P 8100 3850
+F 0 "J?" H 8100 2750 60  0000 C CNN
+F 1 "LCD-S401M16KR" H 8100 4900 60  0000 C CNN
+	1    8100 3850
+	-1   0    0    -1
+$EndComp
+$Comp
+L PIC16LF1933-I/SS U?
+U 1 1 50FF48E1
+P 5550 3950
+F 0 "U?" H 5550 2700 60  0000 C CNN
+F 1 "PIC16LF1933-I/SS" H 5550 5100 60  0000 C CNN
+	1    5550 3950
+	1    0    0    -1
+$EndComp
 $EndSCHEMATC

Commit message: - connect last two lcd pins
Connections:
- wire segments 22 -> 24
Changed lines of the file:
@@
-EESchema Schematic File Version 2  date 1/22/2013 9:40:15 PM
+EESchema Schematic File Version 2  date 2/4/2013 8:52:13 PM
 LIBS:power
 LIBS:device
@@
 LIBS:valves
 LIBS:usb_pwrmon
-LIBS:usb_pwrmon-cache
 EELAYER 25  0
 EELAYER END
@@
 Sheet 1 1
 Title ""
-Date "23 jan 2013"
+Date "5 feb 2013"
 Rev ""
 Comp ""
@@
 Comment4 ""
 $EndDescr
+Wire Wire Line
+	6700 3450 6550 3450
 Wire Wire Line
 	6700 3300 6550 3300
@@
 Wire Wire Line
 	4400 4950 4550 4950
+Wire Wire Line
+	6550 4050 6700 4050
 Text GLabel 4400 3300 0    60   Input ~ 0
 SEG7

Commit message: - add usb ports (will be m/f footprints later).
Parts:
- added J? (x2): USB_NP_1, symbol USB_NP_1
Changed lines of the file:
@@
-EESchema Schematic File Version 2  date 2/4/2013 8:52:13 PM
+EESchema Schematic File Version 2  date 2/22/2013 6:04:26 PM
 LIBS:power
 LIBS:device
@@
 LIBS:valves
 LIBS:usb_pwrmon
+LIBS:usb_pwrmon-cache
 EELAYER 25  0
 EELAYER END
@@
 Sheet 1 1
 Title ""
-Date "5 feb 2013"
+Date "22 feb 2013"
 Rev ""
 Comp ""
@@
 Comment4 ""
 $EndDescr
+$Comp
+L USB_NP_1 J?
+U 1 1 5127F961
+P 9250 3050
+F 0 "J?" H 9250 2500 60  0000 C CNN
+F 1 "USB_NP_1" H 9250 3550 60  0000 C CNN
+	1    9250 3050
+	-1   0    0    1
+$EndComp
+$Comp
+L USB_NP_1 J?
+U 1 1 5127F95A
+P 3150 2700
+F 0 "J?" H 3150 2150 60  0000 C CNN
+F 1 "USB_NP_1" H 3150 3200 60  0000 C CNN
+	1    3150 2700
+	1    0    0    -1
+$EndComp
 Wire Wire Line
-	6700 3450 6550 3450
+	6400 4300 6250 4300
 Wire Wire Line
-	6700 3300 6550 3300
+	6400 4150 6250 4150
 Wire Wire Line
-	4550 4800 4400 4800
+	4250 5650 4100 5650
 Wire Wire Line
-	4550 4200 4400 4200
+	4250 5050 4100 5050
 Wire Wire Line
-	4550 3750 4400 3750
+	4250 4600 4100 4600
 Wire Wire Line
-	4550 3450 4400 3450
+	4250 4300 4100 4300
 Wire Wire Line
-	7700 4700 7550 4700
+	7400 5550 7250 5550
 Wire Wire Line
-	7700 4400 7550 4400
+	7400 5250 7250 5250
 Wire Wire Line
-	7700 4100 7550 4100
+	7400 4950 7250 4950
 Wire Wire Line
-	7700 3800 7550 3800
+	7400 4650 7250 4650
 Wire Wire Line
-	7700 3500 7550 3500
+	7400 4350 7250 4350
 Wire Wire Line
-	7700 3200 7550 3200
+	7400 4050 7250 4050
 Wire Wire Line
-	7550 3050 7700 3050
+	7250 3900 7400 3900
 Wire Wire Line
-	7550 3350 7700 3350
+	7250 4200 7400 4200
 Wire Wire Line
-	7550 3650 7700 3650
+	7250 4500 7400 4500
 Wire Wire Line
-	7550 3950 7700 3950
+	7250 4800 7400 4800
 Wire Wire Line
-	7550 4250 7700 4250
+	7250 5100 7400 5100
 Wire Wire Line
-	7550 4550 7700 4550
+	7250 5400 7400 5400
 Wire Wire Line
-	4400 3300 4550 3300
+	4100 4150 4250 4150
 Wire Wire Line
-	4400 3600 4550 3600
+	4100 4450 4250 4450
 Wire Wire Line
-	4400 3900 4550 3900
+	4100 4750 4250 4750
 Wire Wire Line
-	4400 4350 4550 4350
+	4100 5200 4250 5200
 Wire Wire Line
-	4400 4950 4550 4950
+	4100 5800 4250 5800
 Wire Wire Line
-	6550 4050 6700 4050
-Text GLabel 4400 3300 0    60   Input ~ 0
+	6250 4900 6400 4900
+Text GLabel 4100 4150 0    60   Input ~ 0
 SEG7
-Text GLabel 4400 4950 0    60   Input ~ 0
+Text GLabel 4100 5800 0    60   Input ~ 0
 SEG6
-Text GLabel 4400 3900 0    60   Input ~ 0
+Text GLabel 4100 4750 0    60   Input ~ 0
 SEG5
-Text GLabel 4400 3750 0    60   Input ~ 0
+Text GLabel 4100 4600 0    60   Input ~ 0
 SEG4
-Text GLabel 4400 4800 0    60   Input ~ 0
+Text GLabel 4100 5650 0    60   Input ~ 0
 SEG3
-Text GLabel 4400 4200 0    60   Input ~ 0
+Text GLabel 4100 5050 0    60   Input ~ 0
 SEG2
-Text GLabel 4400 4350 0    60   Input ~ 0
+Text GLabel 4100 5200 0    60   Input ~ 0
 SEG1
-Text GLabel 6700 4050 2    60   Input ~ 0
+Text GLabel 6400 4900 2    60   Input ~ 0
 SEG0
-Text GLabel 4400 3600 0    60   Input ~ 0
+Text GLabel 4100 4450 0    60   Input ~ 0
 COM3
-Text GLabel 4400 3450 0    60   Input ~ 0
+Text GLabel 4100 4300 0    60   Input ~ 0
 COM2
-Text GLabel 6700 3300 2    60   Input ~ 0
+Text GLabel 6400 4150 2    60   Input ~ 0
 COM1
-Text GLabel 6700 3450 2    60   Input ~ 0
+Text GLabel 6400 4300 2    60   Input ~ 0
 COM0
-Text GLabel 7550 4700 0    60   Input ~ 0
+Text GLabel 7250 5550 0    60   Input ~ 0
 SEG7
-Text GLabel 7550 4550 0    60   Input ~ 0
+Text GLabel 7250 5400 0    60   Input ~ 0
 SEG6
-Text GLabel 7550 4400 0    60   Input ~ 0
+Text GLabel 7250 5250 0    60   Input ~ 0
 SEG5
-Text GLabel 7550 4250 0    60   Input ~ 0
+Text GLabel 7250 5100 0    60   Input ~ 0
 SEG4
-Text GLabel 7550 4100 0    60   Input ~ 0
+Text GLabel 7250 4950 0    60   Input ~ 0
 SEG3
-Text GLabel 7550 3950 0    60   Input ~ 0
+Text GLabel 7250 4800 0    60   Input ~ 0
 SEG2
-Text GLabel 7550 3800 0    60   Input ~ 0
+Text GLabel 7250 4650 0    60   Input ~ 0
 SEG1
-Text GLabel 7550 3650 0    60   Input ~ 0
+Text GLabel 7250 4500 0    60   Input ~ 0
 SEG0
-Text GLabel 7550 3500 0    60   Input ~ 0
+Text GLabel 7250 4350 0    60   Input ~ 0
 COM3
-Text GLabel 7550 3350 0    60   Input ~ 0
+Text GLabel 7250 4200 0    60   Input ~ 0
 COM2
-Text GLabel 7550 3200 0    60   Input ~ 0
+Text GLabel 7250 4050 0    60   Input ~ 0
 COM1
-Text GLabel 7550 3050 0    60   Input ~ 0
+Text GLabel 7250 3900 0    60   Input ~ 0
 COM0
 $Comp
 L LCD-S401M16KR J?
 U 1 1 50FF4B2C
-P 8100 3850
-F 0 "J?" H 8100 2750 60  0000 C CNN
-F 1 "LCD-S401M16KR" H 8100 4900 60  0000 C CNN
-	1    8100 3850
+P 7800 4700
+F 0 "J?" H 7800 3600 60  0000 C CNN
+F 1 "LCD-S401M16KR" H 7800 5750 60  0000 C CNN
+	1    7800 4700
 	-1   0    0    -1
 $EndComp
@@
 L PIC16LF1933-I/SS U?
 U 1 1 50FF48E1
-P 5550 3950
-F 0 "U?" H 5550 2700 60  0000 C CNN
-F 1 "PIC16LF1933-I/SS" H 5550 5100 60  0000 C CNN
-	1    5550 3950
+P 5250 4800
+F 0 "U?" H 5250 3550 60  0000 C CNN
+F 1 "PIC16LF1933-I/SS" H 5250 5950 60  0000 C CNN
+	1    5250 4800
 	1    0    0    -1
 $EndComp

Commit message: - add shunt
Parts:
- added R?: R, symbol R
Changed lines of the file:
@@
-EESchema Schematic File Version 2  date 2/22/2013 6:04:26 PM
+EESchema Schematic File Version 2  date 2/22/2013 6:14:41 PM
 LIBS:power
 LIBS:device
@@
 $EndDescr
 $Comp
+L R R?
+U 1 1 5127FAE0
+P 5900 2550
+F 0 "R?" V 5980 2550 50  0000 C CNN
+F 1 "R" V 5900 2550 50  0000 C CNN
+	1    5900 2550
+	0    -1   -1   0
+$EndComp
+$Comp
 L USB_NP_1 J?

Commit message: - add usb ports & connect some gnds.
Parts:
- added J?: USB-MINI, symbol USB-MINI
Connections:
- net labels added: GND
- wire segments 24 -> 34
Other:
- note added: "HOST PC"
- note added: "TARGET DEVICE"
Changed lines of the file:
@@
-EESchema Schematic File Version 2  date 2/22/2013 6:14:41 PM
+EESchema Schematic File Version 2  date 2/23/2013 11:04:50 AM
 LIBS:power
 LIBS:device
@@
 Sheet 1 1
 Title ""
-Date "22 feb 2013"
+Date "23 feb 2013"
 Rev ""
 Comp ""
@@
 Comment4 ""
 $EndDescr
+Wire Wire Line
+	3650 5050 3650 4900
+Wire Wire Line
+	3650 4900 4250 4900
+Wire Wire Line
+	7850 2850 7850 2550
+Wire Wire Line
+	7850 2550 8000 2550
+Connection ~ 2500 2850
+Wire Wire Line
+	2500 3000 2500 2700
+Wire Wire Line
+	2500 2700 2350 2700
+Wire Notes Line
+	9000 1600 9000 3200
+Wire Wire Line
+	6400 4300 6250 4300
+Wire Wire Line
+	6400 4150 6250 4150
+Wire Wire Line
+	4250 5650 4100 5650
+Wire Wire Line
+	4250 5050 4100 5050
+Wire Wire Line
+	4250 4600 4100 4600
+Wire Wire Line
+	4250 4300 4100 4300
+Wire Wire Line
+	7800 5550 7650 5550
+Wire Wire Line
+	7800 5250 7650 5250
+Wire Wire Line
+	7800 4950 7650 4950
+Wire Wire Line
+	7800 4650 7650 4650
+Wire Wire Line
+	7800 4350 7650 4350
+Wire Wire Line
+	7800 4050 7650 4050
+Wire Wire Line
+	7650 3900 7800 3900
+Wire Wire Line
+	7650 4200 7800 4200
+Wire Wire Line
+	7650 4500 7800 4500
+Wire Wire Line
+	7650 4800 7800 4800
+Wire Wire Line
+	7650 5100 7800 5100
+Wire Wire Line
+	7650 5400 7800 5400
+Wire Wire Line
+	4100 4150 4250 4150
+Wire Wire Line
+	4100 4450 4250 4450
+Wire Wire Line
+	4100 4750 4250 4750
+Wire Wire Line
+	4100 5200 4250 5200
+Wire Wire Line
+	4100 5800 4250 5800
+Wire Wire Line
+	6250 4900 6400 4900
+Wire Notes Line
+	1500 1600 1500 5300
+Wire Wire Line
+	2350 2850 2500 2850
+Wire Wire Line
+	2350 4850 2500 4850
+Wire Wire Line
+	2500 4850 2500 5000
+Wire Wire Line
+	8000 2700 7850 2700
+Connection ~ 7850 2700
+$Comp
+L GND #PWR?
+U 1 1 5128E890
+P 3650 5050
+F 0 "#PWR?" H 3650 5050 30  0001 C CNN
+F 1 "GND" H 3650 4980 30  0001 C CNN
+	1    3650 5050
+	1    0    0    -1
+$EndComp
+$Comp
+L GND #PWR?
+U 1 1 5128E871
+P 7850 2850
+F 0 "#PWR?" H 7850 2850 30  0001 C CNN
+F 1 "GND" H 7850 2780 30  0001 C CNN
+	1    7850 2850
+	1    0    0    -1
+$EndComp
+$Comp
+L GND #PWR?
+U 1 1 5128E849
+P 2500 5000
+F 0 "#PWR?" H 2500 5000 30  0001 C CNN
+F 1 "GND" H 2500 4930 30  0001 C CNN
+	1    2500 5000
+	1    0    0    -1
+$EndComp
+$Comp
+L GND #PWR?
+U 1 1 5128E836
+P 2500 3000
+F 0 "#PWR?" H 2500 3000 30  0001 C CNN
+F 1 "GND" H 2500 2930 30  0001 C CNN
+	1    2500 3000
+	1    0    0    -1
+$EndComp
+Text Notes 9100 2400 0    60   ~ 0
+TARGET DEVICE
+Text Notes 1050 3400 0    60   ~ 0
+HOST PC
+$Comp
+L USB-MINI J?
+U 1 1 5128E61E
+P 2050 4550
+F 0 "J?" H 2050 4000 60  0000 C CNN
+F 1 "USB-MINI" H 2050 5100 60  0000 C CNN
+	1    2050 4550
+	1    0    0    -1
+$EndComp
 $Comp
 L R R?
@@
 L USB_NP_1 J?
 U 1 1 5127F961
-P 9250 3050
-F 0 "J?" H 9250 2500 60  0000 C CNN
-F 1 "USB_NP_1" H 9250 3550 60  0000 C CNN
-	1    9250 3050
-	-1   0    0    1
+P 8350 2400
+F 0 "J?" H 8350 1850 60  0000 C CNN
+F 1 "USB_NP_1" H 8350 2900 60  0000 C CNN
+	1    8350 2400
+	-1   0    0    -1
 $EndComp
 $Comp
 L USB_NP_1 J?
 U 1 1 5127F95A
-P 3150 2700
-F 0 "J?" H 3150 2150 60  0000 C CNN
-F 1 "USB_NP_1" H 3150 3200 60  0000 C CNN
-	1    3150 2700
-	1    0    0    -1
-$EndComp
-Wire Wire Line
-	6400 4300 6250 4300
-Wire Wire Line
-	6400 4150 6250 4150
-Wire Wire Line
-	4250 5650 4100 5650
-Wire Wire Line
-	4250 5050 4100 5050
-Wire Wire Line
-	4250 4600 4100 4600
-Wire Wire Line
-	4250 4300 4100 4300
-Wire Wire Line
-	7400 5550 7250 5550
-Wire Wire Line
-	7400 5250 7250 5250
-Wire Wire Line
-	7400 4950 7250 4950
-Wire Wire Line
-	7400 4650 7250 4650
-Wire Wire Line
-	7400 4350 7250 4350
-Wire Wire Line
-	7400 4050 7250 4050
-Wire Wire Line
-	7250 3900 7400 3900
-Wire Wire Line
-	7250 4200 7400 4200
-Wire Wire Line
-	7250 4500 7400 4500
-Wire Wire Line
-	7250 4800 7400 4800
-Wire Wire Line
-	7250 5100 7400 5100
-Wire Wire Line
-	7250 5400 7400 5400
-Wire Wire Line
-	4100 4150 4250 4150
-Wire Wire Line
-	4100 4450 4250 4450
-Wire Wire Line
-	4100 4750 4250 4750
-Wire Wire Line
-	4100 5200 4250 5200
-Wire Wire Line
-	4100 5800 4250 5800
-Wire Wire Line
-	6250 4900 6400 4900
+P 2000 2550
+F 0 "J?" H 2000 2000 60  0000 C CNN
+F 1 "USB_NP_1" H 2000 3050 60  0000 C CNN
+	1    2000 2550
+	1    0    0    -1
+$EndComp
 Text GLabel 4100 4150 0    60   Input ~ 0
 SEG7
@@
 Text GLabel 6400 4300 2    60   Input ~ 0
 COM0
-Text GLabel 7250 5550 0    60   Input ~ 0
+Text GLabel 7650 5550 0    60   Input ~ 0
 SEG7
-Text GLabel 7250 5400 0    60   Input ~ 0
+Text GLabel 7650 5400 0    60   Input ~ 0
 SEG6
-Text GLabel 7250 5250 0    60   Input ~ 0
+Text GLabel 7650 5250 0    60   Input ~ 0
 SEG5
-Text GLabel 7250 5100 0    60   Input ~ 0
+Text GLabel 7650 5100 0    60   Input ~ 0
 SEG4
-Text GLabel 7250 4950 0    60   Input ~ 0
+Text GLabel 7650 4950 0    60   Input ~ 0
 SEG3
-Text GLabel 7250 4800 0    60   Input ~ 0
+Text GLabel 7650 4800 0    60   Input ~ 0
 SEG2
-Text GLabel 7250 4650 0    60   Input ~ 0
+Text GLabel 7650 4650 0    60   Input ~ 0
 SEG1
-Text GLabel 7250 4500 0    60   Input ~ 0
+Text GLabel 7650 4500 0    60   Input ~ 0
 SEG0
-Text GLabel 7250 4350 0    60   Input ~ 0
+Text GLabel 7650 4350 0    60   Input ~ 0
 COM3
-Text GLabel 7250 4200 0    60   Input ~ 0
+Text GLabel 7650 4200 0    60   Input ~ 0
 COM2
-Text GLabel 7250 4050 0    60   Input ~ 0
+Text GLabel 7650 4050 0    60   Input ~ 0
 COM1
-Text GLabel 7250 3900 0    60   Input ~ 0
+Text GLabel 7650 3900 0    60   Input ~ 0
 COM0
 $Comp
 L LCD-S401M16KR J?
 U 1 1 50FF4B2C
-P 7800 4700
-F 0 "J?" H 7800 3600 60  0000 C CNN
-F 1 "LCD-S401M16KR" H 7800 5750 60  0000 C CNN
-	1    7800 4700
+P 8200 4700
+F 0 "J?" H 8200 3600 60  0000 C CNN
+F 1 "LCD-S401M16KR" H 8200 5750 60  0000 C CNN
+	1    8200 4700
 	-1   0    0    -1
 $EndComp

Commit message: - few more pins.
Parts:
- U?: value PIC16LF1933-I/SS -> PIC16F1933-I/SS
Connections:
- net labels added: D+TRGT, D+VCP, D-TRGT, D-VCP, ICSPCLK, ICSPDAT, RX, TX, VBUS, VSENSE
- wire segments 34 -> 54
Other:
- moved on the sheet: R?

Commit message: - add pushbutton for wakeup (portb) and control
Parts:
- added R?: R, symbol R
- added SW?: SW_PUSH, symbol SW_PUSH
Connections:
- net labels added: ADC_SNS
- wire segments 54 -> 60
Changed lines of the file:
@@
-EESchema Schematic File Version 2  date 2/23/2013 11:41:21 AM
+EESchema Schematic File Version 2  date 2/23/2013 11:57:56 AM
 LIBS:power
 LIBS:device
@@
 $EndDescr
 Wire Wire Line
+	10650 5100 10650 4950
+Wire Wire Line
+	10650 4950 10500 4950
+Wire Wire Line
 	2500 4150 2350 4150
 Wire Wire Line
@@
 	2500 4900 2350 4900
 Wire Wire Line
-	9550 5400 9400 5400
-Wire Wire Line
-	9400 5850 9550 5850
-Wire Wire Line
-	9400 4350 9550 4350
+	8850 5700 9000 5700
+Wire Wire Line
+	8850 4200 9000 4200
 Wire Wire Line
 	5100 2350 4950 2350
 Wire Wire Line
 	2350 2550 2500 2550
-Wire Wire Line
-	7250 4200 7400 4200
 Wire Wire Line
 	5100 2050 4800 2050
@@
 	1500 1600 1500 5300
 Wire Wire Line
-	9400 5250 9550 5250
-Wire Wire Line
-	7250 6150 7400 6150
-Wire Wire Line
-	7250 5550 7400 5550
-Wire Wire Line
-	7250 5100 7400 5100
-Wire Wire Line
-	7250 4800 7400 4800
-Wire Wire Line
-	7250 4500 7400 4500
+	8850 5100 9000 5100
+Wire Wire Line
+	6700 6000 6850 6000
+Wire Wire Line
+	6700 5400 6850 5400
+Wire Wire Line
+	6700 4950 6850 4950
+Wire Wire Line
+	6700 4650 6850 4650
+Wire Wire Line
+	6700 4350 6850 4350
 Wire Wire Line
 	8500 2900 8650 2900
@@
 	8650 3050 8500 3050
 Wire Wire Line
-	7400 4650 7250 4650
-Wire Wire Line
-	7400 4950 7250 4950
-Wire Wire Line
-	7400 5400 7250 5400
-Wire Wire Line
-	7400 6000 7250 6000
-Wire Wire Line
-	9550 4500 9400 4500
-Wire Wire Line
-	9550 4650 9400 4650
+	6850 4500 6700 4500
+Wire Wire Line
+	6850 4800 6700 4800
+Wire Wire Line
+	6850 5250 6700 5250
+Wire Wire Line
+	6850 5850 6700 5850
+Wire Wire Line
+	9000 4350 8850 4350
+Wire Wire Line
+	9000 4500 8850 4500
 Wire Notes Line
 	6100 1550 6100 3150
@@
 	4950 2500 4950 2800
 Wire Wire Line
-	7400 5250 6800 5250
-Wire Wire Line
-	6800 5250 6800 5400
+	6850 5100 6250 5100
+Wire Wire Line
+	6250 5100 6250 5250
 Wire Wire Line
 	4950 1900 4950 2050
@@
 	5100 2200 4950 2200
 Wire Wire Line
-	9550 4200 9400 4200
-Wire Wire Line
-	9550 5700 9400 5700
-Wire Wire Line
-	9400 5550 9900 5550
-Wire Wire Line
-	9900 5550 9900 5700
+	9000 4050 8850 4050
+Wire Wire Line
+	9000 5550 8850 5550
+Wire Wire Line
+	8850 5400 9350 5400
+Wire Wire Line
+	9350 5400 9350 5550
 Wire Wire Line
 	2350 4750 2500 4750
@@
 Wire Wire Line
 	2350 4300 2500 4300
+Wire Wire Line
+	9000 4650 8850 4650
+Wire Wire Line
+	6850 4050 6700 4050
+Wire Wire Line
+	9900 5450 9600 5450
+Wire Wire Line
+	9600 5450 9600 5250
+Wire Wire Line
+	9600 5250 8850 5250
+Connection ~ 9750 5450
+Wire Wire Line
+	9900 4950 8850 4950
+Connection ~ 9750 4950
+$Comp
+L GND #PWR?
+U 1 1 5128F432
+P 10650 5100
+F 0 "#PWR?" H 10650 5100 30  0001 C CNN
+F 1 "GND" H 10650 5030 30  0001 C CNN
+	1    10650 5100
+	1    0    0    -1
+$EndComp
+$Comp
+L R R?
+U 1 1 5128F416
+P 9750 5200
+F 0 "R?" V 9830 5200 50  0000 C CNN
+F 1 "R" V 9750 5200 50  0000 C CNN
+	1    9750 5200
+	1    0    0    -1
+$EndComp
+$Comp
+L SW_PUSH SW?
+U 1 1 5128F376
+P 10200 4950
+F 0 "SW?" H 10350 5060 50  0000 C CNN
+F 1 "SW_PUSH" H 10200 4870 50  0000 C CNN
+	1    10200 4950
+	1    0    0    -1
+$EndComp
+Text GLabel 9000 4650 2    60   Input ~ 0
+ADC_SNS
 $Comp
 L GND #PWR?
 U 1 1 5128F037
-P 9900 5700
-F 0 "#PWR?" H 9900 5700 30  0001 C CNN
-F 1 "GND" H 9900 5630 30  0001 C CNN
-	1    9900 5700
-	1    0    0    -1
-$EndComp
-Text GLabel 9550 5400 2    60   Input ~ 0
-VBUS
-Text GLabel 9550 5850 2    60   Input ~ 0
+P 9350 5550
+F 0 "#PWR?" H 9350 5550 30  0001 C CNN
+F 1 "GND" H 9350 5480 30  0001 C CNN
+	1    9350 5550
+	1    0    0    -1
+$EndComp
+Text GLabel 9900 5450 2    60   Input ~ 0
+VBUS
+Text GLabel 9000 5700 2    60   Input ~ 0
 TX
-Text GLabel 9550 5700 2    60   Input ~ 0
+Text GLabel 9000 5550 2    60   Input ~ 0
 RX
-Text GLabel 9550 4350 2    60   Input ~ 0
+Text GLabel 9000 4200 2    60   Input ~ 0
 ICSPCLK
-Text GLabel 9550 4200 2    60   Input ~ 0
+Text GLabel 9000 4050 2    60   Input ~ 0
 ICSPDAT
 Text GLabel 4950 2350 0    60   Input ~ 0
@@
 Text GLabel 2500 2400 2    60   Input ~ 0
 D+TRGT
-Text GLabel 7250 4200 0    60   Input ~ 0
+Text GLabel 6700 4050 0    60   Input ~ 0
 VBUS
 Text GLabel 4950 1900 1    60   Input ~ 0
@@
 L GND #PWR?
 U 1 1 5128E890
-P 6800 5400
-F 0 "#PWR?" H 6800 5400 30  0001 C CNN
-F 1 "GND" H 6800 5330 30  0001 C CNN
-	1    6800 5400
+P 6250 5250
+F 0 "#PWR?" H 6250 5250 30  0001 C CNN
+F 1 "GND" H 6250 5180 30  0001 C CNN
+	1    6250 5250
 	1    0    0    -1
 $EndComp
@@
 	1    0    0    -1
 $EndComp
-Text GLabel 7250 4500 0    60   Input ~ 0
+Text GLabel 6700 4350 0    60   Input ~ 0
 SEG7
-Text GLabel 7250 6150 0    60   Input ~ 0
+Text GLabel 6700 6000 0    60   Input ~ 0
 SEG6
-Text GLabel 7250 5100 0    60   Input ~ 0
+Text GLabel 6700 4950 0    60   Input ~ 0
 SEG5
-Text GLabel 7250 4950 0    60   Input ~ 0
+Text GLabel 6700 4800 0    60   Input ~ 0
 SEG4
-Text GLabel 7250 6000 0    60   Input ~ 0
+Text GLabel 6700 5850 0    60   Input ~ 0
 SEG3
-Text GLabel 7250 5400 0    60   Input ~ 0
+Text GLabel 6700 5250 0    60   Input ~ 0
 SEG2
-Text GLabel 7250 5550 0    60   Input ~ 0
+Text GLabel 6700 5400 0    60   Input ~ 0
 SEG1
-Text GLabel 9550 5250 2    60   Input ~ 0
+Text GLabel 9000 5100 2    60   Input ~ 0
 SEG0
-Text GLabel 7250 4800 0    60   Input ~ 0
+Text GLabel 6700 4650 0    60   Input ~ 0
 COM3
-Text GLabel 7250 4650 0    60   Input ~ 0
+Text GLabel 6700 4500 0    60   Input ~ 0
 COM2
-Text GLabel 9550 4500 2    60   Input ~ 0
+Text GLabel 9000 4350 2    60   Input ~ 0
 COM1
-Text GLabel 9550 4650 2    60   Input ~ 0
+Text GLabel 9000 4500 2    60   Input ~ 0
 COM0
 Text GLabel 8500 3050 0    60   Input ~ 0
@@
 L PIC16LF1933-I/SS U?
 U 1 1 50FF48E1
-P 8400 5150
-F 0 "U?" H 8400 3900 60  0000 C CNN
-F 1 "PIC16F1933-I/SS" H 8400 6300 60  0000 C CNN
-	1    8400 5150
-	1    0    0    -1
-$EndComp
+P 7850 5000
+F 0 "U?" H 7850 3750 60  0000 C CNN
+F 1 "PIC16F1933-I/SS" H 7850 6150 60  0000 C CNN
+	1    7850 5000
+	1    0    0    -1
+$EndComp
