File: hw/kicad/usb_pwrmon.sch (KiCad schematic (older format))
At the start: 12 parts

Commit message: - add ftdi, add decouples for ic vpp
Parts:
- added C?: 0.1uF, symbol C
- added R? (x2): 27R, symbol R
Connections:
- wire segments 65 -> 81
Other:
- moved on the sheet: R?

Commit message: - use OPA378 from ti as instrumentation amp. - add icsp header test points - basic schematic is done at this point
Parts:
- added C?: C, symbol C
- added P? (x5): TX, symbol TST
- added R? (x2): R, symbol R
- added U?: OPA378, symbol OPA378
Connections:
- net labels added: MCLR
- wire segments 81 -> 102
Other:
- moved on the sheet: C?, R?

Commit message: - rename usb connectors
Parts:
- J?: value USB_NP_1 -> USB_A_MALE
- J?: value USB_NP_1 -> USB_A_FEMALE
- J?: value USB-MINI -> USB_MINI_FEMALE
Changed lines of the file:
@@
-EESchema Schematic File Version 2  date 2/24/2013 9:38:18 AM
+EESchema Schematic File Version 2  date 2/24/2013 11:38:50 AM
 LIBS:power
 LIBS:device
@@
 P 1850 3650
 F 0 "J?" H 1850 3100 60  0000 C CNN
-F 1 "USB-MINI" H 1850 4250 60  0000 C CNN
+F 1 "USB_MINI_FEMALE" H 1850 4250 60  0000 C CNN
 	1    1850 3650
 	1    0    0    -1
@@
 P 5700 1750
 F 0 "J?" H 5700 1200 60  0000 C CNN
-F 1 "USB_NP_1" H 5700 2250 60  0000 C CNN
+F 1 "USB_A_FEMALE" H 5700 2250 60  0000 C CNN
 	1    5700 1750
 	-1   0    0    -1
@@
 P 1800 1650
 F 0 "J?" H 1800 1100 60  0000 C CNN
-F 1 "USB_NP_1" H 1800 2150 60  0000 C CNN
+F 1 "USB_A_MALE" H 1800 2150 60  0000 C CNN
 	1    1800 1650
 	1    0    0    -1

Commit message: - NEGATIVE FEEDBACK PLZ >_<
Connections:
- wire segments 102 -> 103

Commit message: - update to low-side current sense. i think this is about done.
Parts:
- removed R?: R, symbol R
- added R? (x2): R, symbol R
Connections:
- net labels added: VLOAD+, VLOAD-
- wire segments 103 -> 98
Other:
- moved on the sheet: C?, R?, SW?

Commit message: - add second gain stage and connect to adc - clean up for drc
Parts:
- added C2: C, symbol C
- added R6, R8, R9: R, symbol R
- added U3: OPA378, symbol OPA378
- gave numbers to parts that had none: 25
Connections:
- net labels added: ADC_SNS_1, ADC_SNS_2
- net labels removed: ADC_SNS
- wire segments 98 -> 114
- no-connect marks 0 -> 14
Other:
- note added: "gain_stage_1"
- note added: "gain_stage_2"
- note added: "shunt"
- moved on the sheet: C1, R3, R4, R5, R7

Commit message: - rename some labels
Parts:
- P1: value TX -> MCLR
- P3: value TX -> VBUS
- P5: value TX -> GND
- P7: value TX -> ICSPDAT
- P8: value TX -> ICSPCLK
Changed lines of the file:
@@
-EESchema Schematic File Version 2  date 3/19/2013 9:47:06 AM
+EESchema Schematic File Version 2  date 8/4/2013 11:18:35 AM
 LIBS:power
 LIBS:device
@@
 Sheet 1 1
 Title ""
-Date "19 mar 2013"
+Date "4 aug 2013"
 Rev ""
 Comp ""
@@
 P 5700 7250
 F 0 "P8" H 5700 7550 40  0000 C CNN
-F 1 "TX" H 5700 7500 30  0000 C CNN
+F 1 "ICSPCLK" H 5700 7500 30  0000 C CNN
 F 2 "" H 5700 7250 60  0001 C CNN
 F 3 "" H 5700 7250 60  0001 C CNN
@@
 P 5550 7100
 F 0 "P7" H 5550 7400 40  0000 C CNN
-F 1 "TX" H 5550 7350 30  0000 C CNN
+F 1 "ICSPDAT" H 5550 7350 30  0000 C CNN
 F 2 "" H 5550 7100 60  0001 C CNN
 F 3 "" H 5550 7100 60  0001 C CNN
@@
 P 5400 6950
 F 0 "P5" H 5400 7250 40  0000 C CNN
-F 1 "TX" H 5400 7200 30  0000 C CNN
+F 1 "GND" H 5400 7200 30  0000 C CNN
 F 2 "" H 5400 6950 60  0001 C CNN
 F 3 "" H 5400 6950 60  0001 C CNN
@@
 P 5250 6800
 F 0 "P3" H 5250 7100 40  0000 C CNN
-F 1 "TX" H 5250 7050 30  0000 C CNN
+F 1 "VBUS" H 5250 7050 30  0000 C CNN
 F 2 "" H 5250 6800 60  0001 C CNN
 F 3 "" H 5250 6800 60  0001 C CNN
@@
 P 5100 6650
 F 0 "P1" H 5100 6950 40  0000 C CNN
-F 1 "TX" H 5100 6900 30  0000 C CNN
+F 1 "MCLR" H 5100 6900 30  0000 C CNN
 F 2 "" H 5100 6650 60  0001 C CNN
 F 3 "" H 5100 6650 60  0001 C CNN

Commit message: - remove everything except one op-amp
Parts:
- removed C2: C, symbol C
- removed C3: 0.1uF, symbol C
- removed J1: USB_A_MALE, symbol USB_NP_1
- removed J2: USB_MINI_FEMALE, symbol USB-MINI
- removed J3: USB_A_FEMALE, symbol USB_NP_1
- removed J4: LCD-S401M16KR, symbol LCD-S401M16KR
- removed P2: TX, symbol TST
- removed P4: RX, symbol TST
- removed P7: ICSPDAT, symbol TST
- removed R1, R2: 27R, symbol R
- removed R10, R6, R8, R9: R, symbol R
- removed SW1: SW_PUSH, symbol SW_PUSH
- removed U1: FT230XS-R, symbol FT230XS-R
- removed U2, U3: OPA378, symbol OPA378
- removed U4: PIC16F1933-I/SS, symbol PIC16LF1933-I/SS
- added R5: R, ~, symbol R
- added U1: AD8591, ~, symbol AD8591
- P1: value MCLR -> VLOAD+
- P3: renamed from P5; value GND -> ADC_IN
- P4: renamed from P8; value ICSPCLK -> VLOAD-
- renumbered P3 to P2, P6 to P8, R3 to R1, R4 to R2, R5 to R3, R7 to R4
Connections:
- net labels added: ADC_IN
- net labels removed: ADC_SNS_2, COM0, COM1, COM2, COM3, D+TRGT, D+VCP, D-TRGT, D-VCP, ICSPCLK, ICSPDAT, MCLR, RX, SEG0, SEG1, SEG2, SEG3, SEG4, SEG5, SEG6, SEG7, TX, VSENSE
- wire segments 114 -> 24
- no-connect marks 14 -> 0
Other:
- note removed: "HOST PC"
- note removed: "NOPOP"
- note removed: "TARGET DEVICE"
- note removed: "gain_stage_1"
- note removed: "gain_stage_2"
- moved on the sheet: C1, R1, R2, R3, R4
