File: hw/kicad/usb_pwrmon.sch (KiCad schematic (older format))
At the start: 12 parts, among them P1 VLOAD+, P2 VBUS, P3 ADC_IN, P4 VLOAD-, P8 GND, U1 AD8591

Commit message: - finish shunt test board
Parts:
- removed R1: R, symbol R
- added R1: LVK12-SHUNT, symbol LVK12-SHUNT
Connections:
- net labels added: VLOAD_MEAS
- net labels removed: ADC_IN
- wire segments 24 -> 28
Changed lines of the file:
@@
-EESchema Schematic File Version 2  date 8/4/2013 11:56:05 AM
+EESchema Schematic File Version 2  date 8/4/2013 12:30:22 PM
 LIBS:power
 LIBS:device
@@
 LIBS:valves
 LIBS:usb_pwrmon
+LIBS:kicadlib
 LIBS:usb_pwrmon-cache
 EELAYER 27 0
@@
 Text GLabel 5550 3700 0    60   Input ~ 0
 VBUS
-$Comp
-L R R1
-U 1 1 513DDCF4
-P 4050 4050
-F 0 "R1" V 4130 4050 50  0000 C CNN
-F 1 "R" V 4050 4050 50  0000 C CNN
-F 2 "" H 4050 4050 60  0001 C CNN
-F 3 "" H 4050 4050 60  0001 C CNN
-	1    4050 4050
-	-1   0    0    1
-$EndComp
-Text GLabel 4050 3700 0    60   Input ~ 0
+Text GLabel 2200 3850 0    60   Input ~ 0
 VLOAD+
-Text GLabel 4050 4400 0    60   Input ~ 0
+Text GLabel 2200 4000 0    60   Input ~ 0
 VLOAD-
 $Comp
 L GND #PWR03
 U 1 1 513DE10D
-P 4450 4600
-F 0 "#PWR03" H 4450 4600 30  0001 C CNN
-F 1 "GND" H 4450 4530 30  0001 C CNN
-F 2 "" H 4450 4600 60  0001 C CNN
-F 3 "" H 4450 4600 60  0001 C CNN
-	1    4450 4600
+P 4150 4600
+F 0 "#PWR03" H 4150 4600 30  0001 C CNN
+F 1 "GND" H 4150 4530 30  0001 C CNN
+F 2 "" H 4150 4600 60  0001 C CNN
+F 3 "" H 4150 4600 60  0001 C CNN
+	1    4150 4600
 	1    0    0    -1
 $EndComp
@@
 Connection ~ 6350 4250
 Wire Wire Line
-	4050 3700 4050 3800
-Wire Wire Line
 	6150 4250 6750 4250
 Wire Wire Line
 	4950 4150 5050 4150
 Text GLabel 4950 4350 0    60   Input ~ 0
-VLOAD+
+VLOAD_MEAS
 Wire Wire Line
 	5050 4350 4950 4350
-Wire Wire Line
-	4450 4150 4450 4600
-Text Notes 3600 4100 0    60   ~ 0
+Text Notes 2800 3600 0    60   ~ 0
 shunt
 Wire Wire Line
@@
 	6600 4800 6350 4800
 Connection ~ 6350 4800
-Wire Wire Line
-	4050 4400 4050 4300
 $Comp
 L AD8591 U1
@@
 	5150 2600 5000 2600
 Text GLabel 4850 2900 2    60   Input ~ 0
-ADC_IN
+ADC_SNS_1
 Wire Wire Line
 	5000 2750 4850 2750
@@
 Wire Wire Line
 	5300 2300 5300 2350
+$Comp
+L LVK12-SHUNT R1
+U 1 1 51FE7DAB
+P 2900 3950
+F 0 "R1" H 2900 3750 60  0000 C CNN
+F 1 "LVK12-SHUNT" H 2900 4150 60  0000 C CNN
+F 2 "" H 2900 3950 60  0000 C CNN
+F 3 "" H 2900 3950 60  0000 C CNN
+	1    2900 3950
+	1    0    0    -1
+$EndComp
+Wire Wire Line
+	2200 3850 2350 3850
+Wire Wire Line
+	2350 4000 2200 4000
+Wire Wire Line
+	4450 4150 4150 4150
+Wire Wire Line
+	4150 4150 4150 4600
+$Comp
+L GND #PWR05
+U 1 1 51FE7ECB
+P 3600 4100
+F 0 "#PWR05" H 3600 4100 30  0001 C CNN
+F 1 "GND" H 3600 4030 30  0001 C CNN
+F 2 "" H 3600 4100 60  0001 C CNN
+F 3 "" H 3600 4100 60  0001 C CNN
+	1    3600 4100
+	1    0    0    -1
+$EndComp
+Wire Wire Line
+	3450 4000 3600 4000
+Text GLabel 3600 3850 2    60   Input ~ 0
+VLOAD_MEAS
+Wire Wire Line
+	3600 3850 3450 3850
+Wire Wire Line
+	3600 4000 3600 4100
 $EndSCHEMATC

Commit message: add max9639
Parts:
- removed R5: R, ~, symbol R
- removed U1: AD8591, ~, symbol AD8591
- added U?: MAX9636, symbol MAX9636
Connections:
- net labels removed: VLOAD_MEAS
- wire segments 28 -> 27
Other:
- moved on the sheet: C1, R1, R2, R4
Changed lines of the file:
@@
-EESchema Schematic File Version 2  date 8/4/2013 12:30:22 PM
+EESchema Schematic File Version 2  date Thu 10 Oct 2013 07:58:54 PM EDT
 LIBS:power
 LIBS:device
@@
 LIBS:valves
 LIBS:usb_pwrmon
-LIBS:kicadlib
 LIBS:usb_pwrmon-cache
-EELAYER 27 0
+EELAYER 25  0
 EELAYER END
-$Descr A4 11693 8268
+$Descr A4 11700 8267
 encoding utf-8
 Sheet 1 1
 Title ""
-Date "4 aug 2013"
+Date "10 oct 2013"
 Rev ""
 Comp ""
@@
 Comment4 ""
 $EndDescr
+Wire Wire Line
+	3900 3850 5050 3850
+Connection ~ 4950 4350
+Wire Wire Line
+	4950 4350 4950 3500
+Wire Wire Line
+	4950 3500 5250 3500
+Wire Wire Line
+	5050 4350 4850 4350
+Connection ~ 6850 4250
+Wire Wire Line
+	6450 4250 7350 4250
+Wire Wire Line
+	6600 4250 6600 3500
+Wire Wire Line
+	6600 3500 5750 3500
+Wire Wire Line
+	5700 3700 6100 3700
+Wire Wire Line
+	5650 4950 5650 4800
+Wire Wire Line
+	6600 4900 6600 4750
+Wire Wire Line
+	4050 4100 4050 4000
+Wire Wire Line
+	4050 4000 3900 4000
+Wire Wire Line
+	2800 4000 2650 4000
+Wire Wire Line
+	2650 3850 2800 3850
+Wire Wire Line
+	5300 2350 5300 2300
+Wire Wire Line
+	4850 2900 4700 2900
+Wire Wire Line
+	5000 2750 4850 2750
+Wire Wire Line
+	5150 2600 5000 2600
+Wire Wire Line
+	5300 2450 5150 2450
+Wire Wire Line
+	5300 2300 5450 2300
+Wire Wire Line
+	6850 4650 6850 4750
+Wire Wire Line
+	6850 4750 6600 4750
+Wire Wire Line
+	5800 4750 5950 4750
+Wire Wire Line
+	5950 4750 5950 3700
+Connection ~ 5950 3700
+Connection ~ 6600 4250
+Wire Wire Line
+	4250 4500 4250 4350
+Wire Wire Line
+	4250 4350 4350 4350
+Wire Wire Line
+	5050 3850 5050 4150
+$Comp
+L MAX9636 U?
+U 1 1 52573E1F
+P 5450 4250
+F 0 "U?" H 5250 4700 60  0000 C CNN
+F 1 "MAX9636" H 5300 3800 60  0000 C CNN
+	1    5450 4250
+	1    0    0    -1
+$EndComp
 $Comp
 L TST P4
@@
 F 0 "P4" H 4850 3050 40  0000 C CNN
 F 1 "VLOAD-" H 4850 3000 30  0000 C CNN
-F 2 "" H 4850 2750 60  0001 C CNN
-F 3 "" H 4850 2750 60  0001 C CNN
 	1    4850 2750
 	1    0    0    -1
@@
 F 0 "P3" H 4700 3200 40  0000 C CNN
 F 1 "ADC_IN" H 4700 3150 30  0000 C CNN
-F 2 "" H 4700 2900 60  0001 C CNN
-F 3 "" H 4700 2900 60  0001 C CNN
 	1    4700 2900
 	1    0    0    -1
@@
 F 0 "P2" H 5150 2750 40  0000 C CNN
 F 1 "VBUS" H 5150 2700 30  0000 C CNN
-F 2 "" H 5150 2450 60  0001 C CNN
-F 3 "" H 5150 2450 60  0001 C CNN
 	1    5150 2450
 	1    0    0    -1
@@
 F 0 "P1" H 5000 2900 40  0000 C CNN
 F 1 "VLOAD+" H 5000 2850 30  0000 C CNN
-F 2 "" H 5000 2600 60  0001 C CNN
-F 3 "" H 5000 2600 60  0001 C CNN
 	1    5000 2600
 	1    0    0    -1
 $EndComp
-Text GLabel 6750 4250 2    60   Input ~ 0
+Text GLabel 7350 4250 2    60   Input ~ 0
 ADC_SNS_1
 $Comp
 L C C1
 U 1 1 512A23CC
-P 6600 4500
-F 0 "C1" H 6650 4600 50  0000 L CNN
-F 1 "C" H 6650 4400 50  0000 L CNN
-F 2 "" H 6600 4500 60  0001 C CNN
-F 3 "" H 6600 4500 60  0001 C CNN
-	1    6600 4500
+P 6850 4450
+F 0 "C1" H 6900 4550 50  0000 L CNN
+F 1 "C" H 6900 4350 50  0000 L CNN
+	1    6850 4450
 	1    0    0    -1
 $EndComp
@@
 L GND #PWR01
 U 1 1 512A235F
-P 5550 5350
-F 0 "#PWR01" H 5550 5350 30  0001 C CNN
-F 1 "GND" H 5550 5280 30  0001 C CNN
-F 2 "" H 5550 5350 60  0001 C CNN
-F 3 "" H 5550 5350 60  0001 C CNN
-	1    5550 5350
+P 5650 4950
+F 0 "#PWR01" H 5650 4950 30  0001 C CNN
+F 1 "GND" H 5650 4880 30  0001 C CNN
+	1    5650 4950
 	1    0    0    -1
 $EndComp
@@
 L R R2
 U 1 1 512A232E
-P 4700 4150
-F 0 "R2" V 4780 4150 50  0000 C CNN
-F 1 "R" V 4700 4150 50  0000 C CNN
-F 2 "" H 4700 4150 60  0001 C CNN
-F 3 "" H 4700 4150 60  0001 C CNN
-	1    4700 4150
+P 4600 4350
+F 0 "R2" V 4680 4350 50  0000 C CNN
+F 1 "R" V 4600 4350 50  0000 C CNN
+	1    4600 4350
 	0    -1   -1   0
 $EndComp
@@
 F 0 "R3" V 5580 3500 50  0000 C CNN
 F 1 "R" V 5500 3500 50  0000 C CNN
-F 2 "" H 5500 3500 60  0001 C CNN
-F 3 "" H 5500 3500 60  0001 C CNN
 	1    5500 3500
 	0    -1   -1   0
@@
 F 0 "P8" H 5300 2600 40  0000 C CNN
 F 1 "GND" H 5300 2550 30  0000 C CNN
-F 2 "" H 5300 2300 60  0001 C CNN
-F 3 "" H 5300 2300 60  0001 C CNN
 	1    5300 2300
 	1    0    0    -1
@@
 L R R4
 U 1 1 513DD91F
-P 6350 4500
-F 0 "R4" V 6430 4500 50  0000 C CNN
-F 1 "R" V 6350 4500 50  0000 C CNN
-F 2 "" H 6350 4500 60  0001 C CNN
-F 3 "" H 6350 4500 60  0001 C CNN
-	1    6350 4500
+P 6600 4500
+F 0 "R4" V 6680 4500 50  0000 C CNN
+F 1 "R" V 6600 4550 50  0000 C CNN
+	1    6600 4500
 	-1   0    0    1
 $EndComp
@@
 L GND #PWR02
 U 1 1 513DD995
-P 6350 4850
-F 0 "#PWR02" H 6350 4850 30  0001 C CNN
-F 1 "GND" H 6350 4780 30  0001 C CNN
-F 2 "" H 6350 4850 60  0001 C CNN
-F 3 "" H 6350 4850 60  0001 C CNN
-	1    6350 4850
-	1    0    0    -1
-$EndComp
-Text GLabel 5550 3700 0    60   Input ~ 0
+P 6600 4900
+F 0 "#PWR02" H 6600 4900 30  0001 C CNN
+F 1 "GND" H 6600 4830 30  0001 C CNN
+	1    6600 4900
+	1    0    0    -1
+$EndComp
+Text GLabel 6100 3700 2    60   Input ~ 0
 VBUS
-Text GLabel 2200 3850 0    60   Input ~ 0
+Text GLabel 2650 3850 0    60   Input ~ 0
 VLOAD+
-Text GLabel 2200 4000 0    60   Input ~ 0
+Text GLabel 2650 4000 0    60   Input ~ 0
 VLOAD-
 $Comp
 L GND #PWR03
 U 1 1 513DE10D
-P 4150 4600
-F 0 "#PWR03" H 4150 4600 30  0001 C CNN
-F 1 "GND" H 4150 4530 30  0001 C CNN
-F 2 "" H 4150 4600 60  0001 C CNN
-F 3 "" H 4150 4600 60  0001 C CNN
-	1    4150 4600
-	1    0    0    -1
-$EndComp
-Wire Wire Line
-	5550 4700 5550 5350
-Wire Wire Line
-	6350 4750 6350 4850
-Wire Wire Line
-	5550 3700 5550 3800
-Connection ~ 6350 4250
-Wire Wire Line
-	6150 4250 6750 4250
-Wire Wire Line
-	4950 4150 5050 4150
-Text GLabel 4950 4350 0    60   Input ~ 0
-VLOAD_MEAS
-Wire Wire Line
-	5050 4350 4950 4350
-Text Notes 2800 3600 0    60   ~ 0
+P 4250 4500
+F 0 "#PWR03" H 4250 4500 30  0001 C CNN
+F 1 "GND" H 4250 4430 30  0001 C CNN
+	1    4250 4500
+	1    0    0    -1
+$EndComp
+Text Notes 3250 3600 0    60   ~ 0
 shunt
-Wire Wire Line
-	5000 4150 5000 3500
-Wire Wire Line
-	5000 3500 5250 3500
-Connection ~ 5000 4150
-Wire Wire Line
-	5750 3500 6350 3500
-Wire Wire Line
-	6350 3500 6350 4250
-Wire Wire Line
-	6600 4300 6600 4250
-Connection ~ 6600 4250
-Wire Wire Line
-	6600 4700 6600 4800
-Wire Wire Line
-	6600 4800 6350 4800
-Connection ~ 6350 4800
-$Comp
-L AD8591 U1
-U 1 1 51FE785A
-P 5350 4250
-F 0 "U1" H 5350 3950 60  0000 C CNN
-F 1 "AD8591" H 5300 4600 60  0000 C CNN
-F 2 "~" H 5350 4250 60  0000 C CNN
-F 3 "~" H 5350 4250 60  0000 C CNN
-	1    5350 4250
-	1    0    0    -1
-$EndComp
-$Comp
-L R R5
-U 1 1 51FE78C0
-P 5650 5000
-F 0 "R5" V 5730 5000 40  0000 C CNN
-F 1 "R" V 5657 5001 40  0000 C CNN
-F 2 "~" V 5580 5000 30  0000 C CNN
-F 3 "~" H 5650 5000 30  0000 C CNN
-	1    5650 5000
-	1    0    0    -1
-$EndComp
-Wire Wire Line
-	5650 5250 5550 5250
-Connection ~ 5550 5250
-Wire Wire Line
-	5650 4750 5650 4650
 Text GLabel 5450 2300 2    60   Input ~ 0
 GND
-Wire Wire Line
-	5450 2300 5300 2300
 Text GLabel 5300 2450 2    60   Input ~ 0
 VBUS
-Wire Wire Line
-	5300 2450 5150 2450
 Text GLabel 5150 2600 2    60   Input ~ 0
 VLOAD+
-Wire Wire Line
-	5150 2600 5000 2600
 Text GLabel 4850 2900 2    60   Input ~ 0
 ADC_SNS_1
-Wire Wire Line
-	5000 2750 4850 2750
-Wire Wire Line
-	4850 2900 4700 2900
 Text GLabel 5000 2750 2    60   Input ~ 0
 VLOAD-
@@
 F 0 "#PWR04" H 5300 2350 30  0001 C CNN
 F 1 "GND" H 5300 2280 30  0001 C CNN
-F 2 "" H 5300 2350 60  0001 C CNN
-F 3 "" H 5300 2350 60  0001 C CNN
 	1    5300 2350
 	1    0    0    -1
 $EndComp
-Wire Wire Line
-	5300 2300 5300 2350
 $Comp
 L LVK12-SHUNT R1
 U 1 1 51FE7DAB
-P 2900 3950
-F 0 "R1" H 2900 3750 60  0000 C CNN
-F 1 "LVK12-SHUNT" H 2900 4150 60  0000 C CNN
-F 2 "" H 2900 3950 60  0000 C CNN
-F 3 "" H 2900 3950 60  0000 C CNN
-	1    2900 3950
-	1    0    0    -1
-$EndComp
-Wire Wire Line
-	2200 3850 2350 3850
-Wire Wire Line
-	2350 4000 2200 4000
-Wire Wire Line
-	4450 4150 4150 4150
-Wire Wire Line
-	4150 4150 4150 4600
+P 3350 3950
+F 0 "R1" H 3350 3750 60  0000 C CNN
+F 1 "LVK12-SHUNT" H 3350 4150 60  0000 C CNN
+	1    3350 3950
+	1    0    0    -1
+$EndComp
 $Comp
 L GND #PWR05
 U 1 1 51FE7ECB
-P 3600 4100
-F 0 "#PWR05" H 3600 4100 30  0001 C CNN
-F 1 "GND" H 3600 4030 30  0001 C CNN
-F 2 "" H 3600 4100 60  0001 C CNN
-F 3 "" H 3600 4100 60  0001 C CNN
-	1    3600 4100
-	1    0    0    -1
-$EndComp
-Wire Wire Line
-	3450 4000 3600 4000
-Text GLabel 3600 3850 2    60   Input ~ 0
-VLOAD_MEAS
-Wire Wire Line
-	3600 3850 3450 3850
-Wire Wire Line
-	3600 4000 3600 4100
+P 4050 4100
+F 0 "#PWR05" H 4050 4100 30  0001 C CNN
+F 1 "GND" H 4050 4030 30  0001 C CNN
+	1    4050 4100
+	1    0    0    -1
+$EndComp
 $EndSCHEMATC

Commit message: save
Parts:
- gave numbers to parts that had none: 1
Changed lines of the file:
@@
-EESchema Schematic File Version 2  date Thu 10 Oct 2013 07:58:54 PM EDT
+EESchema Schematic File Version 2  date Thu 10 Oct 2013 08:25:03 PM EDT
 LIBS:power
 LIBS:device
@@
 Sheet 1 1
 Title ""
-Date "10 oct 2013"
+Date "11 oct 2013"
 Rev ""
 Comp ""
@@
 	5050 3850 5050 4150
 $Comp
-L MAX9636 U?
+L MAX9636 U1
 U 1 1 52573E1F
 P 5450 4250
-F 0 "U?" H 5250 4700 60  0000 C CNN
+F 0 "U1" H 5250 4700 60  0000 C CNN
 F 1 "MAX9636" H 5300 3800 60  0000 C CNN
 	1    5450 4250

Commit message: - fix it all up. ready to roll.
Parts:
- added P5: SHTDN, symbol TST
Connections:
- net labels added: SHTDN
Changed lines of the file:
@@
-EESchema Schematic File Version 2  date Thu 10 Oct 2013 08:25:03 PM EDT
+EESchema Schematic File Version 2  date 10/11/2013 4:06:40 PM
 LIBS:power
 LIBS:device
@@
 LIBS:valves
 LIBS:usb_pwrmon
+LIBS:kicadlib
 LIBS:usb_pwrmon-cache
-EELAYER 25  0
+EELAYER 27 0
 EELAYER END
-$Descr A4 11700 8267
+$Descr A4 11693 8268
 encoding utf-8
 Sheet 1 1
@@
 Wire Wire Line
 	6850 4750 6600 4750
-Wire Wire Line
-	5800 4750 5950 4750
-Wire Wire Line
-	5950 4750 5950 3700
-Connection ~ 5950 3700
 Connection ~ 6600 4250
 Wire Wire Line
@@
 F 0 "U1" H 5250 4700 60  0000 C CNN
 F 1 "MAX9636" H 5300 3800 60  0000 C CNN
+F 2 "" H 5450 4250 60  0001 C CNN
+F 3 "" H 5450 4250 60  0001 C CNN
 	1    5450 4250
 	1    0    0    -1
@@
 F 0 "P4" H 4850 3050 40  0000 C CNN
 F 1 "VLOAD-" H 4850 3000 30  0000 C CNN
+F 2 "" H 4850 2750 60  0001 C CNN
+F 3 "" H 4850 2750 60  0001 C CNN
 	1    4850 2750
 	1    0    0    -1
@@
 F 0 "P3" H 4700 3200 40  0000 C CNN
 F 1 "ADC_IN" H 4700 3150 30  0000 C CNN
+F 2 "" H 4700 2900 60  0001 C CNN
+F 3 "" H 4700 2900 60  0001 C CNN
 	1    4700 2900
 	1    0    0    -1
@@
 F 0 "P2" H 5150 2750 40  0000 C CNN
 F 1 "VBUS" H 5150 2700 30  0000 C CNN
+F 2 "" H 5150 2450 60  0001 C CNN
+F 3 "" H 5150 2450 60  0001 C CNN
 	1    5150 2450
 	1    0    0    -1
@@
 F 0 "P1" H 5000 2900 40  0000 C CNN
 F 1 "VLOAD+" H 5000 2850 30  0000 C CNN
+F 2 "" H 5000 2600 60  0001 C CNN
+F 3 "" H 5000 2600 60  0001 C CNN
 	1    5000 2600
 	1    0    0    -1
@@
 F 0 "C1" H 6900 4550 50  0000 L CNN
 F 1 "C" H 6900 4350 50  0000 L CNN
+F 2 "" H 6850 4450 60  0001 C CNN
+F 3 "" H 6850 4450 60  0001 C CNN
 	1    6850 4450
 	1    0    0    -1
@@
 F 0 "#PWR01" H 5650 4950 30  0001 C CNN
 F 1 "GND" H 5650 4880 30  0001 C CNN
+F 2 "" H 5650 4950 60  0001 C CNN
+F 3 "" H 5650 4950 60  0001 C CNN
 	1    5650 4950
 	1    0    0    -1
@@
 F 0 "R2" V 4680 4350 50  0000 C CNN
 F 1 "R" V 4600 4350 50  0000 C CNN
+F 2 "" H 4600 4350 60  0001 C CNN
+F 3 "" H 4600 4350 60  0001 C CNN
 	1    4600 4350
 	0    -1   -1   0
@@
 F 0 "R3" V 5580 3500 50  0000 C CNN
 F 1 "R" V 5500 3500 50  0000 C CNN
+F 2 "" H 5500 3500 60  0001 C CNN
+F 3 "" H 5500 3500 60  0001 C CNN
 	1    5500 3500
 	0    -1   -1   0
@@
 F 0 "P8" H 5300 2600 40  0000 C CNN
 F 1 "GND" H 5300 2550 30  0000 C CNN
+F 2 "" H 5300 2300 60  0001 C CNN
+F 3 "" H 5300 2300 60  0001 C CNN
 	1    5300 2300
 	1    0    0    -1
@@
 F 0 "R4" V 6680 4500 50  0000 C CNN
 F 1 "R" V 6600 4550 50  0000 C CNN
+F 2 "" H 6600 4500 60  0001 C CNN
+F 3 "" H 6600 4500 60  0001 C CNN
 	1    6600 4500
 	-1   0    0    1
@@
 F 0 "#PWR02" H 6600 4900 30  0001 C CNN
 F 1 "GND" H 6600 4830 30  0001 C CNN
+F 2 "" H 6600 4900 60  0001 C CNN
+F 3 "" H 6600 4900 60  0001 C CNN
 	1    6600 4900
 	1    0    0    -1
@@
 F 0 "#PWR03" H 4250 4500 30  0001 C CNN
 F 1 "GND" H 4250 4430 30  0001 C CNN
+F 2 "" H 4250 4500 60  0001 C CNN
+F 3 "" H 4250 4500 60  0001 C CNN
 	1    4250 4500
 	1    0    0    -1
@@
 F 0 "#PWR04" H 5300 2350 30  0001 C CNN
 F 1 "GND" H 5300 2280 30  0001 C CNN
+F 2 "" H 5300 2350 60  0001 C CNN
+F 3 "" H 5300 2350 60  0001 C CNN
 	1    5300 2350
 	1    0    0    -1
@@
 F 0 "R1" H 3350 3750 60  0000 C CNN
 F 1 "LVK12-SHUNT" H 3350 4150 60  0000 C CNN
+F 2 "" H 3350 3950 60  0001 C CNN
+F 3 "" H 3350 3950 60  0001 C CNN
 	1    3350 3950
 	1    0    0    -1
@@
 F 0 "#PWR05" H 4050 4100 30  0001 C CNN
 F 1 "GND" H 4050 4030 30  0001 C CNN
+F 2 "" H 4050 4100 60  0001 C CNN
+F 3 "" H 4050 4100 60  0001 C CNN
 	1    4050 4100
 	1    0    0    -1
 $EndComp
+Text GLabel 5950 4750 2    60   Input ~ 0
+SHTDN
+Wire Wire Line
+	5950 4750 5800 4750
+Text GLabel 4700 3050 2    60   Input ~ 0
+SHTDN
+$Comp
+L TST P5
+U 1 1 52585AAF
+P 4550 3050
+F 0 "P5" H 4550 3350 40  0000 C CNN
+F 1 "SHTDN" H 4550 3300 30  0000 C CNN
+F 2 "" H 4550 3050 60  0001 C CNN
+F 3 "" H 4550 3050 60  0001 C CNN
+	1    4550 3050
+	1    0    0    -1
+$EndComp
+Wire Wire Line
+	4700 3050 4550 3050
 $EndSCHEMATC

Commit message: new schematic with mkl24/5 and ad8293g80 amp
Parts:
- removed C1: C, symbol C
- removed P1: VLOAD+, symbol TST
- removed P2: VBUS, symbol TST
- removed P3: ADC_IN, symbol TST
- removed P4: VLOAD-, symbol TST
- removed P5: SHTDN, symbol TST
- removed P8: GND, symbol TST
- removed R2, R3, R4: R, symbol R
- removed U1: MAX9636, symbol MAX9636
- added J?: USB_MICRO_B, symbol USB_MICRO_B
- added J?: USB_FEMALE_A, symbol USB_FEMALE_A
- added U?: MKL24Z64VFM4, symbol MKL24Z64VFM4
- added U?: AD8293G80, symbol AD8293G80
Connections:
- net labels added: +5v, D+, D-
- net labels removed: ADC_SNS_1, SHTDN, VBUS, VLOAD+
- wire segments 27 -> 9
Other:
- note removed: "shunt"
- moved on the sheet: R1

Commit message: working on sch
Parts:
- added C?: C, symbol C
- added C?: 2.2uF, symbol C
Connections:
- net +5v: now also U?.6 (VREGIN), C?.1
- net GND: now also C?.2, C?.2
- net +3.3v: now reaches U?.5 (VOUT33)
- net +3.3v: now also C?.1
- no-connect marks 0 -> 1
Changed lines of the file:
@@
 	-1   0    0    1
 $EndComp
+Text GLabel 1650 5300 0    60   Input ~ 0
++5v
+$Comp
+L C C?
+U 1 1 5271BCC1
+P 1750 5600
+F 0 "C?" H 1750 5700 40  0000 L CNN
+F 1 "C" H 1756 5515 40  0000 L CNN
+F 2 "" H 1788 5450 30  0000 C CNN
+F 3 "" H 1750 5600 60  0000 C CNN
+	1    1750 5600
+	1    0    0    -1
+$EndComp
+Wire Wire Line
+	1650 5300 1750 5300
+Wire Wire Line
+	1750 5300 1750 5400
+$Comp
+L GND #PWR?
+U 1 1 5271BCE0
+P 1750 5900
+F 0 "#PWR?" H 1750 5900 30  0001 C CNN
+F 1 "GND" H 1750 5830 30  0001 C CNN
+F 2 "" H 1750 5900 60  0000 C CNN
+F 3 "" H 1750 5900 60  0000 C CNN
+	1    1750 5900
+	1    0    0    -1
+$EndComp
+Wire Wire Line
+	1750 5800 1750 5900
+Text GLabel 5400 3750 0    60   Input ~ 0
++5v
+Wire Wire Line
+	5400 3750 5550 3750
+Text GLabel 5400 3600 0    60   Input ~ 0
++3.3v
+Wire Wire Line
+	5400 3600 5550 3600
+Text GLabel 2200 5300 0    60   Input ~ 0
++3.3v
+$Comp
+L C C?
+U 1 1 5271BD23
+P 2300 5600
+F 0 "C?" H 2300 5700 40  0000 L CNN
+F 1 "2.2uF" H 2306 5515 40  0000 L CNN
+F 2 "" H 2338 5450 30  0000 C CNN
+F 3 "" H 2300 5600 60  0000 C CNN
+	1    2300 5600
+	1    0    0    -1
+$EndComp
+Wire Wire Line
+	2300 5400 2300 5300
+Wire Wire Line
+	2300 5300 2200 5300
+$Comp
+L GND #PWR?
+U 1 1 5271BD3E
+P 2300 5900
+F 0 "#PWR?" H 2300 5900 30  0001 C CNN
+F 1 "GND" H 2300 5830 30  0001 C CNN
+F 2 "" H 2300 5900 60  0000 C CNN
+F 3 "" H 2300 5900 60  0000 C CNN
+	1    2300 5900
+	1    0    0    -1
+$EndComp
+Wire Wire Line
+	2300 5900 2300 5800
+NoConn ~ 1750 3700
 $EndSCHEMATC
