File: hw/kicad/usb_pwrmon.kicad_pcb (KiCad board)
At the start: 2 copper layers, 45.2 x 21.8 mm, 33 parts, among them J1 ARM_10PIN, J2 USB_MALE_A, J3 USB_MICRO_B, J4 USB_FEMALE_A, SW1 SW_PUSH, U1 AD8293G80, U2 MKL24Z64VFM4

Commit message: - change micro b to smt. some more pcb framing.
Former-commit-id: b8d3cdcfd6da06382f3825e487550e1feff4f902
Former-commit-id: efc3568229c1cc02d2fab81a34a9a7aac96a4aff
Former-commit-id: 5ec509d0f138fd51b632a61baea6c092286ae87b
Parts:
- J3: footprint usb_micro_b_10118193-0001LF -> usb_micro_b_smt
- moved U1 13.6 mm to (92.2, 33.5)
- moved JP1 12.9 mm to (66.3, 43.4)
- moved R6 12.2 mm to (94.0, 40.4), turned to 180 degrees
- moved JP2 7.19 mm to (70.6, 45.7)
- moved U2 7.18 mm to (86.9, 30.7)
- moved J_2 4.07 mm to (82.3, 23.9)
- moved SW1 3.82 mm to (102.9, 36.6), turned to 90 degrees
- moved J1 3.70 mm to (99.3, 30.7)
- moved J3 2.05 mm to (83.3, 41.1)
- moved J4 1.05 mm to (114.6, 32.0)
Routing:
- net USB_VBUS: track 12.5 -> 20.8 mm
- net ~RST: track 5.03 -> 0.00 mm
Changed lines of the file:
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@@
   (general
     (links 110)
-    (no_connects 107)
+    (no_connects 108)
     (area 72.060999 21.006999 117.423001 43.001001)
     (thickness 1.6)
     (drawings 4)
-    (tracks 8)
+    (tracks 9)
     (zones 0)
     (modules 33)
@@
   )
   (module sot23-8 (layer F.Cu)
-    (at 81.534 25.146)
+    (at 92.202 33.528)
     (fp_text reference U1 (at 1.651 -1.397) (layer F.SilkS)
       (effects (font (size 0.75 0.75) (thickness 0.12)))
@@
   )
   (module oled_fpc_30 (layer F.Cu)
-    (at 86.36 24.13)
+    (at 82.296 23.876)
     (fp_text reference J_2 (at 0.635 2.54) (layer F.SilkS)
       (effects (font (size 0.75 0.75) (thickness 0.12)))
@@
   )
   (module MKL24Z64VFM4 (layer F.Cu)
-    (at 93.98 31.75 45)
+    (at 86.868 30.734 45)
     (fp_text reference U2 (at -3.771708 -2.334867 45) (layer F.SilkS)
       (effects (font (size 0.75 0.75) (thickness 0.12)))
@@
   )
   (module lvk12 (layer F.Cu)
-    (at 84.074 33.274)
-    (fp_text reference R6 (at 0 -2.032) (layer F.SilkS)
-      (effects (font (size 0.75 0.75) (thickness 0.12)))
-    )
-    (fp_text value LVK12-SHUNT (at 0 -4.1) (layer F.SilkS) hide
+    (at 93.98 40.386 180)
+    (fp_text reference R6 (at -3.302 1.778 180) (layer F.SilkS)
+      (effects (font (size 0.75 0.75) (thickness 0.12)))
+    )
+    (fp_text value LVK12-SHUNT (at 0 -4.1 180) (layer F.SilkS) hide
       (effects (font (size 1.5 1.5) (thickness 0.15)))
     )
-    (pad 1 smd rect (at -1.375 -0.7) (size 1.75 1.1)
+    (pad 1 smd rect (at -1.375 -0.7 180) (size 1.75 1.1)
       (layers F.Cu F.Paste F.Mask)
       (net 32 USB_VBUS)
     )
-    (pad 4 smd rect (at -1.375 0.7) (size 1.75 1.1)
+    (pad 4 smd rect (at -1.375 0.7 180) (size 1.75 1.1)
       (layers F.Cu F.Paste F.Mask)
       (net 15 N-0000037)
     )
-    (pad 2 smd rect (at 1.375 -0.7) (size 1.75 1.1)
+    (pad 2 smd rect (at 1.375 -0.7 180) (size 1.75 1.1)
       (layers F.Cu F.Paste F.Mask)
       (net 32 USB_VBUS)
     )
-    (pad 3 smd rect (at 1.375 0.7) (size 1.75 1.1)
+    (pad 3 smd rect (at 1.375 0.7 180) (size 1.75 1.1)
       (layers F.Cu F.Paste F.Mask)
       (net 15 N-0000037)
@@
   )
   (module jmp_small (layer B.Cu)
-    (at 78.486 39.37)
+    (at 66.294 43.434)
     (fp_text reference JP1 (at 0 2.032) (layer B.SilkS)
       (effects (font (size 0.75 0.75) (thickness 0.12)) (justify mirror))
@@
   )
   (module jmp_small (layer B.Cu)
-    (at 75.438 40.386)
+    (at 70.612 45.72)
     (fp_text reference JP2 (at 0 2.032) (layer B.SilkS)
       (effects (font (size 0.75 0.75) (thickness 0.12)) (justify mirror))
@@
   )
   (module ARM_10_PIN (layer F.Cu)
-    (at 102.87 31.75 180)
+    (at 99.314 30.734 180)
     (fp_text reference J1 (at 0.5 -4 180) (layer F.SilkS)
       (effects (font (size 0.75 0.75) (thickness 0.12)))
@@
   (module usb_a_male_M701-280442 (layer F.Cu)
     (at 74.295 31.115)
-    (fp_text reference J2 (at 3.937 5.207) (layer F.SilkS)
+    (fp_text reference J2 (at 0.381 8.001) (layer F.SilkS)
       (effects (font (size 0.75 0.75) (thickness 0.12)))
     )
@@
     )
   )
-  (module usb_micro_b_10118193-0001LF (layer F.Cu)
-    (at 85.09 40.132)
-    (fp_text reference J3 (at 0 -4.572) (layer F.SilkS)
-      (effects (font (size 0.75 0.75) (thickness 0.12)))
-    )
-    (fp_text value USB_MICRO_B (at 0 2) (layer F.SilkS) hide
-      (effects (font (size 0.75 0.75) (thickness 0.15)))
-    )
-    (pad 5 thru_hole circle (at -3.35 0) (size 2 2) (drill 1.6)
-      (layers *.Cu *.Mask F.SilkS)
-      (net 7 GND)
-    )
-    (pad 5 thru_hole circle (at 3.35 0) (size 2 2) (drill 1.6)
-      (layers *.Cu *.Mask F.SilkS)
-      (net 7 GND)
-    )
-    (pad 5 smd rect (at 1.2 0) (size 0.95 0.95)
-      (layers F.Cu F.Paste F.Mask)
-      (net 7 GND)
-    )
-    (pad 5 smd rect (at -1.2 0) (size 0.95 0.95)
-      (layers F.Cu F.Paste F.Mask)
-      (net 7 GND)
-    )
-    (pad 1 smd rect (at -1.3 -2.675) (size 0.4 1.35)
-      (layers F.Cu F.Paste F.Mask)
-      (net 32 USB_VBUS)
-    )
-    (pad 2 smd rect (at -0.65 -2.675) (size 0.4 1.35)
-      (layers F.Cu F.Paste F.Mask)
-      (net 8 MON_USB_DM)
-    )
-    (pad 3 smd rect (at 0 -2.675) (size 0.4 1.35)
-      (layers F.Cu F.Paste F.Mask)
-      (net 8 MON_USB_DM)
-    )
-    (pad 4 smd rect (at 0.65 -2.675) (size 0.4 1.35)
-      (layers F.Cu F.Paste F.Mask)
-    )
-    (pad 5 smd rect (at 1.3 -2.675) (size 0.4 1.35)
-      (layers F.Cu F.Paste F.Mask)
-      (net 7 GND)
-    )
-    (pad 5 smd rect (at 3.25 -2.5) (size 1.6 1.4)
-      (layers F.Cu F.Paste F.Mask)
-      (net 7 GND)
-    )
-    (pad 5 smd rect (at -3.25 -2.5) (size 1.6 1.4)
-      (layers F.Cu F.Paste F.Mask)
-      (net 7 GND)
-    )
-  )
   (module usb_a_female_87520-0010BLF (layer F.Cu)
-    (at 115.57 31.75 90)
+    (at 114.554 32.004 90)
     (fp_text reference J4 (at -0.012 -4.398 90) (layer F.SilkS)
       (effects (font (size 0.75 0.75) (thickness 0.12)))
@@
   )
   (module spst_pushbutton_smd (layer F.Cu)
-    (at 99.06 36.83)
-    (fp_text reference SW1 (at 0.032 -1.686) (layer F.SilkS)
-      (effects (font (size 0.75 0.75) (thickness 0.12)))
-    )
-    (fp_text value SW_PUSH (at 3.81 6.35) (layer F.SilkS) hide
+    (at 102.87 36.576 90)
+    (fp_text reference SW1 (at 0.032 -1.686 90) (layer F.SilkS)
+      (effects (font (size 0.75 0.75) (thickness 0.12)))
+    )
+    (fp_text value SW_PUSH (at 3.81 6.35 90) (layer F.SilkS) hide
       (effects (font (size 0.75 0.75) (thickness 0.15)))
     )
-    (pad 1 smd rect (at 0 0) (size 1.6 1.4)
-      (layers F.Cu F.Paste F.Mask)
-      (net 7 GND)
-    )
-    (pad 2 smd rect (at 0 4.5) (size 1.6 1.4)
+    (pad 1 smd rect (at 0 0 90) (size 1.6 1.4)
+      (layers F.Cu F.Paste F.Mask)
+      (net 7 GND)
+    )
+    (pad 2 smd rect (at 0 4.5 90) (size 1.6 1.4)
       (layers F.Cu F.Paste F.Mask)
       (net 13 N-0000020)
     )
-    (pad 1 smd rect (at 8.4 0) (size 1.6 1.4)
-      (layers F.Cu F.Paste F.Mask)
-      (net 7 GND)
-    )
-    (pad 2 smd rect (at 8.4 4.5) (size 1.6 1.4)
+    (pad 1 smd rect (at 8.4 0 90) (size 1.6 1.4)
+      (layers F.Cu F.Paste F.Mask)
+      (net 7 GND)
+    )
+    (pad 2 smd rect (at 8.4 4.5 90) (size 1.6 1.4)
       (layers F.Cu F.Paste F.Mask)
       (net 13 N-0000020)
@@
       (layers F.Cu F.Paste F.Mask)
       (net 29 TRGT_USB_DM)
+    )
+  )
+  (module usb_micro_b_smt (layer F.Cu)
+    (at 83.312 41.148)
+    (fp_text reference J3 (at 5.334 -2.032) (layer F.SilkS)
+      (effects (font (size 0.75 0.75) (thickness 0.12)))
+    )
+    (fp_text value USB_MICRO_B (at 0 2.159) (layer F.SilkS) hide
+      (effects (font (size 0.75 0.75) (thickness 0.15)))
+    )
+    (pad 6 smd rect (at 1.2 0) (size 1.9 1.9)
+      (layers F.Cu F.Paste F.Mask)
+      (net 7 GND)
+    )
+    (pad 6 smd rect (at -1.2 0) (size 1.9 1.9)
+      (layers F.Cu F.Paste F.Mask)
+      (net 7 GND)
+    )
+    (pad 6 smd rect (at 3.8 0) (size 1.8 1.9)
+      (layers F.Cu F.Paste F.Mask)
+      (net 7 GND)
+    )
+    (pad 6 smd rect (at -3.8 0) (size 1.8 1.9)
+      (layers F.Cu F.Paste F.Mask)
+      (net 7 GND)
+    )
+    (pad 6 smd rect (at -3.1 -2.55) (size 2.1 1.6)
+      (layers F.Cu F.Paste F.Mask)
+      (net 7 GND)
+    )
+    (pad 6 smd rect (at 3.1 -2.55) (size 2.1 1.6)
+      (layers F.Cu F.Paste F.Mask)
+      (net 7 GND)
+    )
+    (pad 2 smd rect (at -0.65 -3) (size 0.4 2)
+      (layers F.Cu F.Paste F.Mask)
+      (net 8 MON_USB_DM)
+    )
+    (pad 3 smd rect (at 0 -3) (size 0.4 2)
+      (layers F.Cu F.Paste F.Mask)
+      (net 8 MON_USB_DM)
+    )
+    (pad 4 smd rect (at 0.65 -3) (size 0.4 2)
+      (layers F.Cu F.Paste F.Mask)
+    )
+    (pad 5 smd rect (at 1.3 -3) (size 0.4 2)
+      (layers F.Cu F.Paste F.Mask)
+      (net 7 GND)
+    )
+    (pad 1 smd rect (at -1.3 -3) (size 0.4 2)
+      (layers F.Cu F.Paste F.Mask)
+      (net 32 USB_VBUS)
     )
   )
@@
   (gr_line (start 117.348 21.082) (end 117.348 42.926) (angle 90) (layer Edge.Cuts) (width 0.15))
   (gr_line (start 72.136 21.082) (end 117.348 21.082) (angle 90) (layer Edge.Cuts) (width 0.15))
-  (segment (start 83.79 37.457) (end 83.79 36.546) (width 0.5) (layer F.Cu) (net 32))
-  (segment (start 79.494 35.814) (end 78.295 34.615) (width 0.5) (layer F.Cu) (net 32))
-  (segment (start 83.058 35.814) (end 79.494 35.814) (width 0.5) (layer F.Cu) (net 32))
-  (segment (start 83.79 36.546) (end 83.058 35.814) (width 0.5) (layer F.Cu) (net 32))
-  (segment (start 78.295 34.615) (end 80.336 32.574) (width 0.5) (layer F.Cu) (net 32))
-  (segment (start 80.336 32.574) (end 82.699 32.574) (width 0.5) (layer F.Cu) (net 32))
-  (segment (start 94.492652 28.762474) (end 95.46 27.795126) (width 0.254) (layer F.Cu) (net 34))
-  (segment (start 95.46 27.795126) (end 95.46 24.13) (width 0.254) (layer F.Cu) (net 34))
+  (segment (start 92.605 41.086) (end 90.87 41.086) (width 0.5) (layer F.Cu) (net 32))
+  (segment (start 90.87 41.086) (end 89.916 40.132) (width 0.5) (layer F.Cu) (net 32))
+  (segment (start 81.026 35.814) (end 87.376 35.814) (width 0.5) (layer F.Cu) (net 32))
+  (segment (start 89.916 38.354) (end 89.916 40.132) (width 0.5) (layer F.Cu) (net 32))
+  (segment (start 87.376 35.814) (end 89.916 38.354) (width 0.5) (layer F.Cu) (net 32))
+  (segment (start 79.494 35.814) (end 81.026 35.814) (width 0.5) (layer F.Cu) (net 32))
+  (segment (start 78.295 34.615) (end 79.494 35.814) (width 0.5) (layer F.Cu) (net 32))
+  (segment (start 82.012 36.8) (end 82.012 38.148) (width 0.5) (layer F.Cu) (net 32))
+  (segment (start 81.026 35.814) (end 82.012 36.8) (width 0.5) (layer F.Cu) (net 32))
 )
